File: kicad/Chess.kicad_sch (KiCad schematic)
At the start: 71 parts, among them J1 Raspberry_Pi_2_3, U1 CD74HC4067M, U12 A1302xUA, U13 A1302xUA, U14 A1302xUA, U15 A1302xUA, U16 A1302xUA, U17 A1302xUA, U18 A1302xUA, U19 A1302xUA, U2 ADS1015IDGS, U20 A1302xUA, U21 A1302xUA, U22 A1302xUA, U23 A1302xUA, U24 A1302xUA, U25 A1302xUA, U26 A1302xUA, U27 A1302xUA, U28 A1302xUA, U29 A1302xUA, U3 AMS1117, U30 A1302xUA, U31 A1302xUA, U32 A1302xUA, U33 A1302xUA, U34 A1302xUA, U35 A1302xUA, U36 A1302xUA, U37 A1302xUA, U38 A1302xUA, U39 A1302xUA, U4 CD74HC4067M, U40 A1302xUA, U41 A1302xUA, U42 A1302xUA, U43 A1302xUA, U44 A1302xUA, U45 A1302xUA, U46 A1302xUA, U47 A1302xUA, U48 A1302xUA, U49 A1302xUA, U5 CD74HC4067M, U50 A1302xUA, U51 A1302xUA, U52 A1302xUA, U53 A1302xUA, U54 A1302xUA, U55 A1302xUA, U56 A1302xUA, U57 A1302xUA, U58 A1302xUA, U59 A1302xUA, U6 CD74HC4067M, U60 A1302xUA, U61 A1302xUA, U62 A1302xUA, U63 A1302xUA, U64 A1302xUA, U65 A1302xUA, U66 A1302xUA, U67 A1302xUA, U68 A1302xUA, U69 A1302xUA, U70 A1302xUA, U71 A1302xUA, U72 A1302xUA, U73 A1302xUA, U74 A1302xUA, U75 A1302xUA

Commit message: labels
Parts:
- removed U3: AMS1117, Package_TO_SOT_SMD:SOT-223-3_TabPin2, symbol Regulator_Linear:AMS1117
- added U3: MP1584EN, Package_TO_SOT_SMD:SOT-223-3_TabPin2, symbol New_Library:MP1584EN
- J1: now left out of the parts list
Connections:
- net 3.3V: now also U3.3 (OUT+)
- net 5V: now also U3.1 (IN+)
- net GND: now also U3.2 (IN-), U3.4 (OUT-); no longer U2.3 (GND), U6.12 (GND)
Other:
- moved on the sheet: U2

Commit message: sensors
Parts:
- U12, U13, U14, U15, U16, U17, U18, U19, U20, U21, U22, U23, U24, U25, U26, U27, U28, U29, U30, U31, U32, U33, U34, U35, U36, U37, U38, U39, U40, U41, U42, U43, U44, U45, U46, U47, U48, U49, U50, U51, U52, U53, U54, U55, U56, U57, U58, U59, U60, U61, U62, U63, U64, U65, U66, U67, U68, U69, U70, U71, U72, U73, U74, U75: footprint Package_TO_SOT_THT:TO-92S -> SEN3_SS49E_HNW; symbol Sensor_Magnetic:A1302xUA -> SS49E:SS49E
Connections:
- net GND: now also U12.3 (OUT), U13.3 (OUT), U14.3 (OUT), U15.3 (OUT), U16.3 (OUT), U17.3 (OUT), U18.3 (OUT), U19.3 (OUT), U20.3 (OUT), U21.3 (OUT), U22.3 (OUT), U23.3 (OUT), U24.3 (OUT), U25.3 (OUT), U26.3 (OUT), U27.3 (OUT), U28.3 (OUT), U29.3 (OUT), U30.3 (OUT), U31.3 (OUT), U32.3 (OUT), U33.3 (OUT), U34.3 (OUT), U35.3 (OUT), U36.3 (OUT), U37.3 (OUT), U38.3 (OUT), U39.3 (OUT), U40.3 (OUT), U41.3 (OUT), U42.3 (OUT), U43.3 (OUT), U44.3 (OUT), U45.3 (OUT), U46.3 (OUT), U47.3 (OUT), U48.3 (OUT), U49.3 (OUT), U50.3 (OUT), U51.3 (OUT), U52.3 (OUT), U53.3 (OUT), U54.3 (OUT), U55.3 (OUT), U56.3 (OUT), U57.3 (OUT), U58.3 (OUT), U59.3 (OUT), U60.3 (OUT), U61.3 (OUT), U62.3 (OUT), U63.3 (OUT), U64.3 (OUT), U65.3 (OUT), U66.3 (OUT), U67.3 (OUT), U68.3 (OUT), U69.3 (OUT), U70.3 (OUT), U71.3 (OUT), U72.3 (OUT), U73.3 (OUT), U74.3 (OUT), U75.3 (OUT); no longer U12.2 (GND), U13.2 (GND), U14.2 (GND), U15.2 (GND), U16.2 (GND), U17.2 (GND), U18.2 (GND), U19.2 (GND), U20.2 (GND), U21.2 (GND), U22.2 (GND), U23.2 (GND), U24.2 (GND), U25.2 (GND), U26.2 (GND), U27.2 (GND), U28.2 (GND), U29.2 (GND), U30.2 (GND), U31.2 (GND), U32.2 (GND), U33.2 (GND), U34.2 (GND), U35.2 (GND), U36.2 (GND), U37.2 (GND), U38.2 (GND), U39.2 (GND), U40.2 (GND), U41.2 (GND), U42.2 (GND), U43.2 (GND), U44.2 (GND), U45.2 (GND), U46.2 (GND), U47.2 (GND), U48.2 (GND), U49.2 (GND), U50.2 (GND), U51.2 (GND), U52.2 (GND), U53.2 (GND), U54.2 (GND), U55.2 (GND), U56.2 (GND), U57.2 (GND), U58.2 (GND), U59.2 (GND), U60.2 (GND), U61.2 (GND), U62.2 (GND), U63.2 (GND), U64.2 (GND), U65.2 (GND), U66.2 (GND), U67.2 (GND), U68.2 (GND), U69.2 (GND), U70.2 (GND), U71.2 (GND), U72.2 (GND), U73.2 (GND), U74.2 (GND), U75.2 (GND)

Commit message: sensor connections
Connections:
- net GND: now also U6.12 (GND)
- net MD13: now reaches U50.2 (GND)
- net MD13: now also U5.19 (I12)
- net MA12: now reaches U37.2 (GND)
- net MA12: now also U6.20 (I11)
- net MC12: now reaches U73.2 (GND)
- net MC12: now also U4.5 (I4)
- net MB12: now reaches U61.2 (GND)
- net MB12: now also U1.5 (I4)
- net MC1: now reaches U4.16 (I15)
- net MC1: now also U68.2 (GND)
- net MC2: now reaches U4.17 (I14)
- net MC2: now also U67.2 (GND)
- net MC3: now reaches U4.18 (I13)
- net MC3: now also U45.2 (GND)
- net MC4: now reaches U4.19 (I12)
- net MC4: now also U42.2 (GND)
- net MC9: now reaches U4.2 (I7)
- net MC9: now also U72.2 (GND)
- net MC5: now reaches U4.20 (I11)
- net MC5: now also U64.2 (GND)
- net MC6: now reaches U4.21 (I10)
- net MC6: now also U65.2 (GND)
- net MC7: now reaches U4.22 (I9)
- net MC7: now also U66.2 (GND)
- net MC8: now reaches U4.23 (I8)
- net MC8: now also U69.2 (GND)
- net MC10: now reaches U4.3 (I6)
- net MC10: now also U75.2 (GND)
- net MC11: now reaches U4.4 (I5)
- net MC11: now also U74.2 (GND)
- net MC13: now reaches U4.6 (I3)
- net MC13: now also U51.2 (GND)
- net MC14: now reaches U4.7 (I2)
- net MC14: now also U48.2 (GND)
- net MC15: now reaches U4.8 (I1)
- net MC15: now also U70.2 (GND)
- net MC16: now reaches U4.9 (I0)
- net MC16: now also U71.2 (GND)
- net MD10: now reaches U19.2 (GND)
- net MD10: now also U5.22 (I9)
- net MA8: now reaches U13.2 (GND)
- net MA8: now also U6.2 (I7)
- net MD15: now reaches U46.2 (GND)
- net MD15: now also U5.17 (I14)
- net MD11: now reaches U27.2 (GND)
- net MD11: now also U5.21 (I10)
- net MA5: now reaches U28.2 (GND)
- net MA5: now also U6.5 (I4)
- net MB2: now reaches U55.2 (GND)
- net MB2: now also U1.17 (I14)
- net MA11: now reaches U23.2 (GND)
- net MA11: now also U6.21 (I10)
- net MD9: now reaches U18.2 (GND)
- net MD9: now also U5.23 (I8)
- net MB7: now reaches U54.2 (GND)
- net MB7: now also U1.22 (I9)
- net MB1: now reaches U56.2 (GND)
- net MB1: now also U1.16 (I15)
- net MB8: now reaches U57.2 (GND)
- net MB8: now also U1.23 (I8)
- net MB10: now reaches U63.2 (GND)
- net MB10: now also U1.3 (I6)
- net MA16: now reaches U6.16 (I15)
- net MA16: now also U22.2 (GND)
- net MA15: now reaches U6.17 (I14)
- net MA15: now also U34.2 (GND)
- net MA14: now reaches U6.18 (I13)
- net MA14: now also U35.2 (GND)
- net MA13: now reaches U6.19 (I12)
- net MA13: now also U38.2 (GND)
- net MA10: now reaches U6.22 (I9)
- net MA10: now also U15.2 (GND)
- net MA9: now reaches U6.23 (I8)
- net MA9: now also U14.2 (GND)
- net MA7: now reaches U6.3 (I6)
- net MA7: now also U12.2 (GND)
- net MA6: now reaches U6.4 (I5)
- net MA6: now also U20.2 (GND)
- net MA4: now reaches U6.6 (I3)
- net MA4: now also U29.2 (GND)
- net MA3: now reaches U6.7 (I2)
- net MA3: now also U32.2 (GND)
- net MA2: now reaches U6.8 (I1)
- net MA2: now also U31.2 (GND)
- net MA1: now reaches U6.9 (I0)
- net MA1: now also U21.2 (GND)
- net MB4: now reaches U30.2 (GND)
- net MB4: now also U1.19 (I12)
- net MB9: now reaches U60.2 (GND)
- net MB9: now also U1.2 (I7)
- net MD8: now reaches U17.2 (GND)
- net MD8: now also U5.2 (I7)
- net MD16: now reaches U26.2 (GND)
- net MD16: now also U5.16 (I15)
- net MB5: now reaches U52.2 (GND)
- net MB5: now also U1.20 (I11)
- net MB15: now reaches U58.2 (GND)
- net MB15: now also U1.8 (I1)
- net MD14: now reaches U47.2 (GND)
- net MD14: now also U5.18 (I13)
- net MB6: now reaches U53.2 (GND)
- net MB6: now also U1.21 (I10)
- net MD3: now reaches U44.2 (GND)
- net MD3: now also U5.7 (I2)
- net MB16: now reaches U59.2 (GND)
- net MB16: now also U1.9 (I0)
- net MD4: now reaches U41.2 (GND)
- net MD4: now also U5.6 (I3)
- net MD12: now reaches U49.2 (GND)
- net MD12: now also U5.20 (I11)
- net MD6: now reaches U24.2 (GND)
- net MD6: now also U5.4 (I5)
- net MB14: now reaches U36.2 (GND)
- net MB14: now also U1.7 (I2)
- net MD5: now reaches U40.2 (GND)
- net MD5: now also U5.5 (I4)
- net MB3: now reaches U33.2 (GND)
- net MB3: now also U1.18 (I13)
- net MD1: now reaches U25.2 (GND)
- net MD1: now also U5.9 (I0)
- net MB13: now reaches U39.2 (GND)
- net MB13: now also U1.6 (I3)
- net MD2: now reaches U43.2 (GND)
- net MD2: now also U5.8 (I1)
- net MB11: now reaches U1.4 (I5)
- net MB11: now also U62.2 (GND)
- net MD7: now reaches U5.3 (I6)
- net MD7: now also U16.2 (GND)
Other:
- moved on the sheet: J1, U1, U12, U13, U14, U15, U16, U17, U18, U19, U2, U20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

Commit message: libraries
Parts:
- U12, U13, U14, U15, U16, U17, U18, U19, U20, U21, U22, U23, U24, U25, U26, U27, U28, U29, U30, U31, U32, U33, U34, U35, U36, U37, U38, U39, U40, U41, U42, U43, U44, U45, U46, U47, U48, U49, U50, U51, U52, U53, U54, U55, U56, U57, U58, U59, U60, U61, U62, U63, U64, U65, U66, U67, U68, U69, U70, U71, U72, U73, U74, U75: symbol SS49E:SS49E -> MagChess:SS49E
- U3: symbol New_Library:MP1584EN -> MagChess:MP1584EN
Changed lines of the file:
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@@
 	)
 	(symbol
-		(lib_id "SS49E:SS49E")
+		(lib_id "MagChess:SS49E")
 		(at 203.2 237.49 0)
 		(unit 1)
@@
 	)
 	(symbol
-		(lib_id "SS49E:SS49E")
+		(lib_id "MagChess:SS49E")
 		(at 228.6 151.13 0)
 		(unit 1)
@@
 	)
 	(symbol
-		(lib_id "SS49E:SS49E")
+		(lib_id "MagChess:SS49E")
 		(at 152.4 237.49 0)
 		(unit 1)
@@
 	)
 	(symbol
-		(lib_id "SS49E:SS49E")
+		(lib_id "MagChess:SS49E")
 		(at 152.4 151.13 0)
 		(unit 1)
@@
 	)
 	(symbol
-		(lib_id "SS49E:SS49E")
+		(lib_id "MagChess:SS49E")
 		(at 152.4 215.9 0)
 		(unit 1)
@@
 	)
 	(symbol
-		(lib_id "SS49E:SS49E")
+		(lib_id "MagChess:SS49E")
 		(at 279.4 237.49 0)
 		(unit 1)
@@
 	)
 	(symbol
-		(lib_id "SS49E:SS49E")
+		(lib_id "MagChess:SS49E")
 		(at 279.4 107.95 0)
 		(unit 1)
@@
 	)
 	(symbol
-		(lib_id "SS49E:SS49E")
+		(lib_id "MagChess:SS49E")
 		(at 228.6 215.9 0)
 		(unit 1)
@@
 	)
 	(symbol
-		(lib_id "SS49E:SS49E")
+		(lib_id "MagChess:SS49E")
 		(at 152.4 194.31 0)
 		(unit 1)
@@
 	)
 	(symbol
-		(lib_id "SS49E:SS49E")
+		(lib_id "MagChess:SS49E")
 		(at 254 237.49 0)
 		(unit 1)
@@
 	)
 	(symbol
-		(lib_id "SS49E:SS49E")
+		(lib_id "MagChess:SS49E")
 		(at 228.6 86.36 0)
 		(unit 1)
@@
 	)
 	(symbol
-		(lib_id "SS49E:SS49E")
+		(lib_id "MagChess:SS49E")
 		(at 152.4 107.95 0)
 		(unit 1)
@@
 	)
 	(symbol
-		(lib_id "SS49E:SS49E")
+		(lib_id "MagChess:SS49E")
 		(at 254 151.13 0)
 		(unit 1)
@@
 	)
 	(symbol
-		(lib_id "SS49E:SS49E")
+		(lib_id "MagChess:SS49E")
 		(at 279.4 215.9 0)
 		(unit 1)
@@
 	)
 	(symbol
-		(lib_id "SS49E:SS49E")
+		(lib_id "MagChess:SS49E")
 		(at 101.6 86.36 0)
 		(unit 1)
@@
 	)
 	(symbol
-		(lib_id "SS49E:SS49E")
+		(lib_id "MagChess:SS49E")
 		(at 127 107.95 0)
 		(unit 1)
@@
 	)
 	(symbol
-		(lib_id "SS49E:SS49E")
+		(lib_id "MagChess:SS49E")
 		(at 127 215.9 0)
 		(unit 1)
@@
 	)
 	(symbol
-		(lib_id "SS49E:SS49E")
+		(lib_id "MagChess:SS49E")
 		(at 127 194.31 0)
 		(unit 1)
@@
 	)
 	(symbol
-		(lib_id "SS49E:SS49E")
+		(lib_id "MagChess:SS49E")
 		(at 101.6 107.95 0)
 		(unit 1)
@@
 	)
 	(symbol
-		(lib_id "SS49E:SS49E")
+		(lib_id "MagChess:SS49E")
 		(at 177.8 237.49 0)
 		(unit 1)
@@
 	)
 	(symbol
-		(lib_id "SS49E:SS49E")
+		(lib_id "MagChess:SS49E")
 		(at 101.6 194.31 0)
 		(unit 1)
@@
 	)
 	(symbol
-		(lib_id "SS49E:SS49E")
+		(lib_id "MagChess:SS49E")
 		(at 101.6 151.13 0)
 		(unit 1)
@@
 	)
 	(symbol
-		(lib_id "SS49E:SS49E")
+		(lib_id "MagChess:SS49E")
 		(at 177.8 86.36 0)
 		(unit 1)
@@
 	)
 	(symbol
-		(lib_id "SS49E:SS49E")
+		(lib_id "MagChess:SS49E")
 		(at 101.6 129.54 0)
 		(unit 1)
@@
 	)
 	(symbol
-		(lib_id "SS49E:SS49E")
+		(lib_id "MagChess:SS49E")
 		(at 279.4 194.31 0)
 		(unit 1)
@@
 	)
 	(symbol
-		(lib_id "SS49E:SS49E")
+		(lib_id "MagChess:SS49E")
 		(at 228.6 129.54 0)
 		(unit 1)
@@
 	)
 	(symbol
-		(lib_id "SS49E:SS49E")
+		(lib_id "MagChess:SS49E")
 		(at 254 215.9 0)
 		(unit 1)
@@
 	)
 	(symbol
-		(lib_id "SS49E:SS49E")
+		(lib_id "MagChess:SS49E")
 		(at 152.4 86.36 0)
 		(unit 1)
@@
 	)
 	(symbol
-		(lib_id "SS49E:SS49E")
+		(lib_id "MagChess:SS49E")
 		(at 152.4 129.54 0)
 		(unit 1)
@@
 	)
 	(symbol
-		(lib_id "SS49E:SS49E")
+		(lib_id "MagChess:SS49E")
 		(at 279.4 129.54 0)
 		(unit 1)
@@
 	)
 	(symbol
-		(lib_id "SS49E:SS49E")
+		(lib_id "MagChess:SS49E")
 		(at 203.2 215.9 0)
 		(unit 1)
@@
 	)
 	(symbol
-		(lib_id "SS49E:SS49E")
+		(lib_id "MagChess:SS49E")
 		(at 127 86.36 0)
 		(unit 1)
@@
 	)
 	(symbol
-		(lib_id "SS49E:SS49E")
+		(lib_id "MagChess:SS49E")
 		(at 279.4 151.13 0)
 		(unit 1)
@@
 	)
 	(symbol
-		(lib_id "SS49E:SS49E")
+		(lib_id "MagChess:SS49E")
 		(at 203.2 107.95 0)
 		(unit 1)
@@
 	)
 	(symbol
-		(lib_id "SS49E:SS49E")
+		(lib_id "MagChess:SS49E")
 		(at 203.2 194.31 0)
 		(unit 1)
@@
 	)
 	(symbol
-		(lib_id "SS49E:SS49E")
+		(lib_id "MagChess:SS49E")
 		(at 127 129.54 0)
 		(unit 1)
@@
 	)
 	(symbol
-		(lib_id "SS49E:SS49E")
+		(lib_id "MagChess:SS49E")
 		(at 177.8 172.72 0)
 		(unit 1)
@@
 	)
 	(symbol
-		(lib_id "SS49E:SS49E")
+		(lib_id "MagChess:SS49E")
 		(at 101.6 215.9 0)
 		(unit 1)
@@
 	)
 	(symbol
-		(lib_id "SS49E:SS49E")
+		(lib_id "MagChess:SS49E")
 		(at 127 237.49 0)
 		(unit 1)
@@
 	)
 	(symbol
-		(lib_id "SS49E:SS49E")
+		(lib_id "MagChess:SS49E")
 		(at 254 86.36 0)
 		(unit 1)
@@
 	)
 	(symbol
-		(lib_id "SS49E:SS49E")
+		(lib_id "MagChess:SS49E")
 		(at 203.2 172.72 0)
 		(unit 1)
@@
 	)
 	(symbol
-		(lib_id "SS49E:SS49E")
+		(lib_id "MagChess:SS49E")
 		(at 228.6 237.49 0)
 		(unit 1)
@@
 	)
 	(symbol
-		(lib_id "SS49E:SS49E")
+		(lib_id "MagChess:SS49E")
 		(at 101.6 172.72 0)
 		(unit 1)
@@
 	)
 	(symbol
-		(lib_id "SS49E:SS49E")
+		(lib_id "MagChess:SS49E")
 		(at 254 172.72 0)
 		(unit 1)
@@
 	)
 	(symbol
-		(lib_id "SS49E:SS49E")
+		(lib_id "MagChess:SS49E")
 		(at 254 107.95 0)
 		(unit 1)
@@
 	)
 	(symbol
-		(lib_id "SS49E:SS49E")
+		(lib_id "MagChess:SS49E")
 		(at 177.8 215.9 0)
 		(unit 1)
@@
 	)
 	(symbol
-		(lib_id "SS49E:SS49E")
+		(lib_id "MagChess:SS49E")
 		(at 177.8 129.54 0)
 		(unit 1)
@@
 	)
 	(symbol
-		(lib_id "SS49E:SS49E")
+		(lib_id "MagChess:SS49E")
 		(at 127 172.72 0)
 		(unit 1)
@@
 	)
 	(symbol
-		(lib_id "SS49E:SS49E")
+		(lib_id "MagChess:SS49E")
 		(at 177.8 194.31 0)
 		(unit 1)
@@
 	)
 	(symbol
-		(lib_id "SS49E:SS49E")
+		(lib_id "MagChess:SS49E")
 		(at 228.6 172.72 0)
 		(unit 1)
@@
 	)
 	(symbol
-		(lib_id "SS49E:SS49E")
+		(lib_id "MagChess:SS49E")
 		(at 152.4 172.72 0)
 		(unit 1)
@@
 	)
 	(symbol
-		(lib_id "SS49E:SS49E")
+		(lib_id "MagChess:SS49E")
 		(at 177.8 107.95 0)
 		(unit 1)
@@
 	)
 	(symbol
-		(lib_id "SS49E:SS49E")
+		(lib_id "MagChess:SS49E")
 		(at 254 194.31 0)
 		(unit 1)
@@
 	)
 	(symbol
-		(lib_id "SS49E:SS49E")
+		(lib_id "MagChess:SS49E")
 		(at 101.6 237.49 0)
 		(unit 1)
@@
 	)
 	(symbol
-		(lib_id "SS49E:SS49E")
+		(lib_id "MagChess:SS49E")
 		(at 177.8 151.13 0)
 		(unit 1)
@@
 	)
 	(symbol
-		(lib_id "SS49E:SS49E")
+		(lib_id "MagChess:SS49E")
 		(at 228.6 194.31 0)
 		(unit 1)
@@
 	)
 	(symbol
-		(lib_id "SS49E:SS49E")
+		(lib_id "MagChess:SS49E")
 		(at 203.2 151.13 0)
 		(unit 1)
@@
 	)
 	(symbol
-		(lib_id "SS49E:SS49E")
+		(lib_id "MagChess:SS49E")
 		(at 127 151.13 0)
 		(unit 1)
@@
 	)
 	(symbol
-		(lib_id "SS49E:SS49E")
+		(lib_id "MagChess:SS49E")
 		(at 203.2 129.54 0)
 		(unit 1)
@@
 	)
 	(symbol
-		(lib_id "SS49E:SS49E")
+		(lib_id "MagChess:SS49E")
 		(at 279.4 86.36 0)
 		(unit 1)
@@
 	)
 	(symbol
-		(lib_id "SS49E:SS49E")
+		(lib_id "MagChess:SS49E")
 		(at 203.2 86.36 0)
 		(unit 1)
@@
 	)
 	(symbol
-		(lib_id "SS49E:SS49E")
+		(lib_id "MagChess:SS49E")
 		(at 254 129.54 0)
 		(unit 1)
@@
 	)
 	(symbol
-		(lib_id "SS49E:SS49E")
+		(lib_id "MagChess:SS49E")
 		(at 279.4 172.72 0)
 		(unit 1)
@@
 	)
 	(symbol
-		(lib_id "New_Library:MP1584EN")
+		(lib_id "MagChess:MP1584EN")
 		(at 398.78 231.14 0)
 		(unit 1)
@@
 	)
 	(symbol
-		(lib_id "SS49E:SS49E")
+		(lib_id "MagChess:SS49E")
 		(at 228.6 107.95 0)
 		(unit 1)

Commit message: libraries
Parts:
- U12, U13, U14, U15, U16, U17, U18, U19, U20, U21, U22, U23, U24, U25, U26, U27, U28, U29, U30, U31, U32, U33, U34, U35, U36, U37, U38, U39, U40, U41, U42, U43, U44, U45, U46, U47, U48, U49, U50, U51, U52, U53, U54, U55, U56, U57, U58, U59, U60, U61, U62, U63, U64, U65, U66, U67, U68, U69, U70, U71, U72, U73, U74, U75: footprint SEN3_SS49E_HNW -> MagChess Footprints:SS49E
Changed lines of the file:
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@@
 			)
 		)
-		(property "Footprint" "SEN3_SS49E_HNW"
+		(property "Footprint" "MagChess Footprints:SS49E"
 			(at 203.2 237.49 0)
 			(effects
@@
 			)
 		)
-		(property "Footprint" "SEN3_SS49E_HNW"
+		(property "Footprint" "MagChess Footprints:SS49E"
 			(at 228.6 151.13 0)
 			(effects
@@
 			)
 		)
-		(property "Footprint" "SEN3_SS49E_HNW"
+		(property "Footprint" "MagChess Footprints:SS49E"
 			(at 152.4 237.49 0)
 			(effects
@@
 			)
 		)
-		(property "Footprint" "SEN3_SS49E_HNW"
+		(property "Footprint" "MagChess Footprints:SS49E"
 			(at 152.4 151.13 0)
 			(effects
@@
 			)
 		)
-		(property "Footprint" "SEN3_SS49E_HNW"
+		(property "Footprint" "MagChess Footprints:SS49E"
 			(at 152.4 215.9 0)
 			(effects
@@
 			)
 		)
-		(property "Footprint" "SEN3_SS49E_HNW"
+		(property "Footprint" "MagChess Footprints:SS49E"
 			(at 279.4 237.49 0)
 			(effects
@@
 			)
 		)
-		(property "Footprint" "SEN3_SS49E_HNW"
+		(property "Footprint" "MagChess Footprints:SS49E"
 			(at 279.4 107.95 0)
 			(effects
@@
 			)
 		)
-		(property "Footprint" "SEN3_SS49E_HNW"
+		(property "Footprint" "MagChess Footprints:SS49E"
 			(at 228.6 215.9 0)
 			(effects
@@
 			)
 		)
-		(property "Footprint" "SEN3_SS49E_HNW"
+		(property "Footprint" "MagChess Footprints:SS49E"
 			(at 152.4 194.31 0)
 			(effects
@@
 			)
 		)
-		(property "Footprint" "SEN3_SS49E_HNW"
+		(property "Footprint" "MagChess Footprints:SS49E"
 			(at 254 237.49 0)
 			(effects
@@
 			)
 		)
-		(property "Footprint" "SEN3_SS49E_HNW"
+		(property "Footprint" "MagChess Footprints:SS49E"
 			(at 228.6 86.36 0)
 			(effects
@@
 			)
 		)
-		(property "Footprint" "SEN3_SS49E_HNW"
+		(property "Footprint" "MagChess Footprints:SS49E"
 			(at 152.4 107.95 0)
 			(effects
@@
 			)
 		)
-		(property "Footprint" "SEN3_SS49E_HNW"
+		(property "Footprint" "MagChess Footprints:SS49E"
 			(at 254 151.13 0)
 			(effects
@@
 			)
 		)
-		(property "Footprint" "SEN3_SS49E_HNW"
+		(property "Footprint" "MagChess Footprints:SS49E"
 			(at 279.4 215.9 0)
 			(effects
@@
 			)
 		)
-		(property "Footprint" "SEN3_SS49E_HNW"
+		(property "Footprint" "MagChess Footprints:SS49E"
 			(at 101.6 86.36 0)
 			(effects
@@
 			)
 		)
-		(property "Footprint" "SEN3_SS49E_HNW"
+		(property "Footprint" "MagChess Footprints:SS49E"
 			(at 127 107.95 0)
 			(effects
@@
 			)
 		)
-		(property "Footprint" "SEN3_SS49E_HNW"
+		(property "Footprint" "MagChess Footprints:SS49E"
 			(at 127 215.9 0)
 			(effects
@@
 			)
 		)
-		(property "Footprint" "SEN3_SS49E_HNW"
+		(property "Footprint" "MagChess Footprints:SS49E"
 			(at 127 194.31 0)
 			(effects
@@
 			)
 		)
-		(property "Footprint" "SEN3_SS49E_HNW"
+		(property "Footprint" "MagChess Footprints:SS49E"
 			(at 101.6 107.95 0)
 			(effects
@@
 			)
 		)
-		(property "Footprint" "SEN3_SS49E_HNW"
+		(property "Footprint" "MagChess Footprints:SS49E"
 			(at 177.8 237.49 0)
 			(effects
@@
 			)
 		)
-		(property "Footprint" "SEN3_SS49E_HNW"
+		(property "Footprint" "MagChess Footprints:SS49E"
 			(at 101.6 194.31 0)
 			(effects
@@
 			)
 		)
-		(property "Footprint" "SEN3_SS49E_HNW"
+		(property "Footprint" "MagChess Footprints:SS49E"
 			(at 101.6 151.13 0)
 			(effects
@@
 			)
 		)
-		(property "Footprint" "SEN3_SS49E_HNW"
+		(property "Footprint" "MagChess Footprints:SS49E"
 			(at 177.8 86.36 0)
 			(effects
@@
 			)
 		)
-		(property "Footprint" "SEN3_SS49E_HNW"
+		(property "Footprint" "MagChess Footprints:SS49E"
 			(at 101.6 129.54 0)
 			(effects
@@
 			)
 		)
-		(property "Footprint" "SEN3_SS49E_HNW"
+		(property "Footprint" "MagChess Footprints:SS49E"
 			(at 279.4 194.31 0)
 			(effects
@@
 			)
 		)
-		(property "Footprint" "SEN3_SS49E_HNW"
+		(property "Footprint" "MagChess Footprints:SS49E"
 			(at 228.6 129.54 0)
 			(effects
@@
 			)
 		)
-		(property "Footprint" "SEN3_SS49E_HNW"
+		(property "Footprint" "MagChess Footprints:SS49E"
 			(at 254 215.9 0)
 			(effects
@@
 			)
 		)
-		(property "Footprint" "SEN3_SS49E_HNW"
+		(property "Footprint" "MagChess Footprints:SS49E"
 			(at 152.4 86.36 0)
 			(effects
@@
 			)
 		)
-		(property "Footprint" "SEN3_SS49E_HNW"
+		(property "Footprint" "MagChess Footprints:SS49E"
 			(at 152.4 129.54 0)
 			(effects
@@
 			)
 		)
-		(property "Footprint" "SEN3_SS49E_HNW"
+		(property "Footprint" "MagChess Footprints:SS49E"
 			(at 279.4 129.54 0)
 			(effects
@@
 			)
 		)
-		(property "Footprint" "SEN3_SS49E_HNW"
+		(property "Footprint" "MagChess Footprints:SS49E"
 			(at 203.2 215.9 0)
 			(effects
@@
 			)
 		)
-		(property "Footprint" "SEN3_SS49E_HNW"
+		(property "Footprint" "MagChess Footprints:SS49E"
 			(at 127 86.36 0)
 			(effects
@@
 			)
 		)
-		(property "Footprint" "SEN3_SS49E_HNW"
+		(property "Footprint" "MagChess Footprints:SS49E"
 			(at 279.4 151.13 0)
 			(effects
@@
 			)
 		)
-		(property "Footprint" "SEN3_SS49E_HNW"
+		(property "Footprint" "MagChess Footprints:SS49E"
 			(at 203.2 107.95 0)
 			(effects
@@
 			)
 		)
-		(property "Footprint" "SEN3_SS49E_HNW"
+		(property "Footprint" "MagChess Footprints:SS49E"
 			(at 203.2 194.31 0)
 			(effects
@@
 			)
 		)
-		(property "Footprint" "SEN3_SS49E_HNW"
+		(property "Footprint" "MagChess Footprints:SS49E"
 			(at 127 129.54 0)
 			(effects
@@
 			)
 		)
-		(property "Footprint" "SEN3_SS49E_HNW"
+		(property "Footprint" "MagChess Footprints:SS49E"
 			(at 177.8 172.72 0)
 			(effects
@@
 			)
 		)
-		(property "Footprint" "SEN3_SS49E_HNW"
+		(property "Footprint" "MagChess Footprints:SS49E"
 			(at 101.6 215.9 0)
 			(effects
@@
 			)
 		)
-		(property "Footprint" "SEN3_SS49E_HNW"
+		(property "Footprint" "MagChess Footprints:SS49E"
 			(at 127 237.49 0)
 			(effects
@@
 			)
 		)
-		(property "Footprint" "SEN3_SS49E_HNW"
+		(property "Footprint" "MagChess Footprints:SS49E"
 			(at 254 86.36 0)
 			(effects
@@
 			)
 		)
-		(property "Footprint" "SEN3_SS49E_HNW"
+		(property "Footprint" "MagChess Footprints:SS49E"
 			(at 203.2 172.72 0)
 			(effects
@@
 			)
 		)
-		(property "Footprint" "SEN3_SS49E_HNW"
+		(property "Footprint" "MagChess Footprints:SS49E"
 			(at 228.6 237.49 0)
 			(effects
@@
 			)
 		)
-		(property "Footprint" "SEN3_SS49E_HNW"
+		(property "Footprint" "MagChess Footprints:SS49E"
 			(at 101.6 172.72 0)
 			(effects
@@
 			)
 		)
-		(property "Footprint" "SEN3_SS49E_HNW"
+		(property "Footprint" "MagChess Footprints:SS49E"
 			(at 254 172.72 0)
 			(effects
@@
 			)
 		)
-		(property "Footprint" "SEN3_SS49E_HNW"
+		(property "Footprint" "MagChess Footprints:SS49E"
 			(at 254 107.95 0)
 			(effects
@@
 			)
 		)
-		(property "Footprint" "SEN3_SS49E_HNW"
+		(property "Footprint" "MagChess Footprints:SS49E"
 			(at 177.8 215.9 0)
 			(effects
@@
 			)
 		)
-		(property "Footprint" "SEN3_SS49E_HNW"
+		(property "Footprint" "MagChess Footprints:SS49E"
 			(at 177.8 129.54 0)
 			(effects
@@
 			)
 		)
-		(property "Footprint" "SEN3_SS49E_HNW"
+		(property "Footprint" "MagChess Footprints:SS49E"
 			(at 127 172.72 0)
 			(effects
@@
 			)
 		)
-		(property "Footprint" "SEN3_SS49E_HNW"
+		(property "Footprint" "MagChess Footprints:SS49E"
 			(at 177.8 194.31 0)
 			(effects
@@
 			)
 		)
-		(property "Footprint" "SEN3_SS49E_HNW"
+		(property "Footprint" "MagChess Footprints:SS49E"
 			(at 228.6 172.72 0)
 			(effects
@@
 			)
 		)
-		(property "Footprint" "SEN3_SS49E_HNW"
+		(property "Footprint" "MagChess Footprints:SS49E"
 			(at 152.4 172.72 0)
 			(effects
@@
 			)
 		)
-		(property "Footprint" "SEN3_SS49E_HNW"
+		(property "Footprint" "MagChess Footprints:SS49E"
 			(at 177.8 107.95 0)
 			(effects
@@
 			)
 		)
-		(property "Footprint" "SEN3_SS49E_HNW"
+		(property "Footprint" "MagChess Footprints:SS49E"
 			(at 254 194.31 0)
 			(effects
@@
 			)
 		)
-		(property "Footprint" "SEN3_SS49E_HNW"
+		(property "Footprint" "MagChess Footprints:SS49E"
 			(at 101.6 237.49 0)
 			(effects
@@
 			)
 		)
-		(property "Footprint" "SEN3_SS49E_HNW"
+		(property "Footprint" "MagChess Footprints:SS49E"
 			(at 177.8 151.13 0)
 			(effects
@@
 			)
 		)
-		(property "Footprint" "SEN3_SS49E_HNW"
+		(property "Footprint" "MagChess Footprints:SS49E"
 			(at 228.6 194.31 0)
 			(effects
@@
 			)
 		)
-		(property "Footprint" "SEN3_SS49E_HNW"
+		(property "Footprint" "MagChess Footprints:SS49E"
 			(at 203.2 151.13 0)
 			(effects
@@
 			)
 		)
-		(property "Footprint" "SEN3_SS49E_HNW"
+		(property "Footprint" "MagChess Footprints:SS49E"
 			(at 127 151.13 0)
 			(effects
@@
 			)
 		)
-		(property "Footprint" "SEN3_SS49E_HNW"
+		(property "Footprint" "MagChess Footprints:SS49E"
 			(at 203.2 129.54 0)
 			(effects
@@
 			)
 		)
-		(property "Footprint" "SEN3_SS49E_HNW"
+		(property "Footprint" "MagChess Footprints:SS49E"
 			(at 279.4 86.36 0)
 			(effects
@@
 			)
 		)
-		(property "Footprint" "SEN3_SS49E_HNW"
+		(property "Footprint" "MagChess Footprints:SS49E"
 			(at 203.2 86.36 0)
 			(effects
@@
 			)
 		)
-		(property "Footprint" "SEN3_SS49E_HNW"
+		(property "Footprint" "MagChess Footprints:SS49E"
 			(at 254 129.54 0)
 			(effects
@@
 			)
 		)
-		(property "Footprint" "SEN3_SS49E_HNW"
+		(property "Footprint" "MagChess Footprints:SS49E"
 			(at 279.4 172.72 0)
 			(effects
@@
 			)
 		)
-		(property "Footprint" "SEN3_SS49E_HNW"
+		(property "Footprint" "MagChess Footprints:SS49E"
 			(at 228.6 107.95 0)
 			(effects

Commit message: update
Parts:
- removed J1: Raspberry_Pi_2_3, symbol Connector:Raspberry_Pi_2_3
- added J2: Conn_01x08_Pin, Connector_PinHeader_2.54mm:PinHeader_1x08_P2.54mm_Vertical, symbol Connector:Conn_01x08_Pin
Connections:
- net 5V: now also J2.1 (Pin_1)
- net GND: now also U2.3 (GND), J2.8 (Pin_8)
- net S0: now also J2.2 (Pin_2)
- net S1: now also J2.3 (Pin_3)
- net S2: now also J2.4 (Pin_4)
- net S3: now also J2.5 (Pin_5)
- net SCL: now also J2.6 (Pin_6)
- net SDA: now also J2.7 (Pin_7)
Other:
- moved on the sheet: U1, U12, U13, U14, U15, U16, U17, U18, U19, U2, U20, U21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
