File: kicad/Chess.kicad_sch (KiCad schematic)
At the start: 71 parts, among them J2 Conn_01x08_Pin, U1 CD74HC4067M, U12 A1302xUA, U13 A1302xUA, U14 A1302xUA, U15 A1302xUA, U16 A1302xUA, U17 A1302xUA, U18 A1302xUA, U19 A1302xUA, U2 ADS1015IDGS, U20 A1302xUA, U21 A1302xUA, U22 A1302xUA, U23 A1302xUA, U24 A1302xUA, U25 A1302xUA, U26 A1302xUA, U27 A1302xUA, U28 A1302xUA, U29 A1302xUA, U3 MP1584EN, U30 A1302xUA, U31 A1302xUA, U32 A1302xUA, U33 A1302xUA, U34 A1302xUA, U35 A1302xUA, U36 A1302xUA, U37 A1302xUA, U38 A1302xUA, U39 A1302xUA, U4 CD74HC4067M, U40 A1302xUA, U41 A1302xUA, U42 A1302xUA, U43 A1302xUA, U44 A1302xUA, U45 A1302xUA, U46 A1302xUA, U47 A1302xUA, U48 A1302xUA, U49 A1302xUA, U5 CD74HC4067M, U50 A1302xUA, U51 A1302xUA, U52 A1302xUA, U53 A1302xUA, U54 A1302xUA, U55 A1302xUA, U56 A1302xUA, U57 A1302xUA, U58 A1302xUA, U59 A1302xUA, U6 CD74HC4067M, U60 A1302xUA, U61 A1302xUA, U62 A1302xUA, U63 A1302xUA, U64 A1302xUA, U65 A1302xUA, U66 A1302xUA, U67 A1302xUA, U68 A1302xUA, U69 A1302xUA, U70 A1302xUA, U71 A1302xUA, U72 A1302xUA, U73 A1302xUA, U74 A1302xUA, U75 A1302xUA

Commit message: MP1584 2
Parts:
- U3: footprint Package_TO_SOT_SMD:SOT-223-3_TabPin2 -> MagChess Footprints:MP1584
Changed lines of the file:
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@@
 			)
 		)
-		(property "Footprint" "Package_TO_SOT_SMD:SOT-223-3_TabPin2"
+		(property "Footprint" "MagChess Footprints:MP1584"
 			(at 407.67 229.87 0)
 			(effects
@@
 			)
 		)
-		(property "Datasheet" "http://www.diodes.com/datasheets/AP1117.pdf"
+		(property "Datasheet" ""
 			(at 410.21 241.3 0)
 			(effects
@@
 			)
 		)
-		(property "Description" "1A Low Dropout regulator, positive, adjustable output, SOT-223"
+		(property "Description" ""
 			(at 407.67 234.95 0)
 			(effects

Commit message: routes 2
Connections:
- net SCL: now also J2.7 (Pin_7); no longer J2.6 (Pin_6)
- net SDA: now also J2.6 (Pin_6); no longer J2.7 (Pin_7)
- net at U4.1 (COM): now also U2.7 (AIN3); no longer U2.6 (AIN2)
- net at U5.1 (COM): now also U2.6 (AIN2); no longer U2.7 (AIN3)
Changed lines of the file:
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@@
 	(wire
 		(pts
+			(xy 378.46 242.57) (xy 353.06 242.57)
+		)
+		(stroke
+			(width 0)
+			(type default)
+		)
+	)
+	(wire
+		(pts
 			(xy 158.75 139.7) (xy 158.75 161.29)
 		)
@@
 	(wire
 		(pts
-			(xy 379.73 185.42) (xy 389.89 185.42)
-		)
-		(stroke
-			(width 0)
-			(type default)
-		)
-	)
-	(wire
-		(pts
 			(xy 260.35 226.06) (xy 260.35 247.65)
 		)
@@
 	(wire
 		(pts
+			(xy 382.27 185.42) (xy 389.89 185.42)
+		)
+		(stroke
+			(width 0)
+			(type default)
+		)
+	)
+	(wire
+		(pts
 			(xy 87.63 226.06) (xy 87.63 247.65)
 		)
@@
 	(wire
 		(pts
-			(xy 379.73 242.57) (xy 379.73 185.42)
+			(xy 379.73 245.11) (xy 379.73 187.96)
 		)
 		(stroke
@@
 	(wire
 		(pts
+			(xy 378.46 245.11) (xy 378.46 242.57)
+		)
+		(stroke
+			(width 0)
+			(type default)
+		)
+	)
+	(wire
+		(pts
 			(xy 113.03 182.88) (xy 113.03 204.47)
 		)
@@
 	(wire
 		(pts
-			(xy 240.03 139.7) (xy 240.03 161.29)
+			(xy 382.27 185.42) (xy 382.27 214.63)
 		)
 		(stroke
@@
 	(wire
 		(pts
-			(xy 184.15 118.11) (xy 184.15 139.7)
+			(xy 240.03 139.7) (xy 240.03 161.29)
 		)
 		(stroke
@@
 	(wire
 		(pts
-			(xy 163.83 161.29) (xy 163.83 182.88)
+			(xy 184.15 118.11) (xy 184.15 139.7)
 		)
 		(stroke
@@
 	(wire
 		(pts
-			(xy 382.27 187.96) (xy 389.89 187.96)
+			(xy 163.83 161.29) (xy 163.83 182.88)
 		)
 		(stroke
@@
 	(wire
 		(pts
-			(xy 382.27 214.63) (xy 382.27 187.96)
-		)
-		(stroke
-			(width 0)
-			(type default)
-		)
-	)
-	(wire
-		(pts
 			(xy 265.43 226.06) (xy 265.43 247.65)
 		)
@@
 	(wire
 		(pts
+			(xy 379.73 187.96) (xy 389.89 187.96)
+		)
+		(stroke
+			(width 0)
+			(type default)
+		)
+	)
+	(wire
+		(pts
 			(xy 285.75 247.65) (xy 285.75 269.24)
 		)
@@
 	(wire
 		(pts
-			(xy 353.06 242.57) (xy 379.73 242.57)
+			(xy 378.46 245.11) (xy 379.73 245.11)
 		)
 		(stroke
@@
 	(global_label "SCL"
 		(shape input)
-		(at 400.05 269.24 90)
+		(at 402.59 269.24 90)
 		(fields_autoplaced yes)
 		(effects
@@
 		)
 		(property "Intersheetrefs" "${INTERSHEET_REFS}"
-			(at 400.05 262.7472 90)
+			(at 402.59 262.7472 90)
 			(effects
 				(font
@@
 	(global_label "SDA"
 		(shape input)
-		(at 402.59 269.24 90)
+		(at 400.05 269.24 90)
 		(fields_autoplaced yes)
 		(effects
@@
 		)
 		(property "Intersheetrefs" "${INTERSHEET_REFS}"
-			(at 402.59 262.6867 90)
+			(at 400.05 262.6867 90)
 			(effects
 				(font

Commit message: routing v2
Connections:
- net MA1: now also U6.4 (I5); no longer U6.9 (I0)
- net MA11: now also U6.16 (I15); no longer U6.21 (I10)
- net MA12: now also U6.17 (I14); no longer U6.20 (I11)
- net MA13: now also U6.18 (I13); no longer U6.19 (I12)
- net MA14: now also U6.19 (I12); no longer U6.18 (I13)
- net MA15: now also U6.20 (I11); no longer U6.17 (I14)
- net MA16: now also U6.21 (I10); no longer U6.16 (I15)
- net MA2: now also U6.5 (I4); no longer U6.8 (I1)
- net MA3: now also U6.6 (I3); no longer U6.7 (I2)
- net MA4: now also U6.7 (I2); no longer U6.6 (I3)
- net MA5: now also U6.8 (I1); no longer U6.5 (I4)
- net MA6: now also U6.9 (I0); no longer U6.4 (I5)
- net MB1: now also U1.21 (I10); no longer U1.16 (I15)
- net MB11: now also U1.9 (I0); no longer U1.4 (I5)
- net MB12: now also U1.8 (I1); no longer U1.5 (I4)
- net MB13: now also U1.7 (I2); no longer U1.6 (I3)
- net MB14: now also U1.6 (I3); no longer U1.7 (I2)
- net MB15: now also U1.5 (I4); no longer U1.8 (I1)
- net MB16: now also U1.4 (I5); no longer U1.9 (I0)
- net MB2: now also U1.20 (I11); no longer U1.17 (I14)
- net MB3: now also U1.19 (I12); no longer U1.18 (I13)
- net MB4: now also U1.18 (I13); no longer U1.19 (I12)
- net MB5: now also U1.17 (I14); no longer U1.20 (I11)
- net MB6: now also U1.16 (I15); no longer U1.21 (I10)
- net MC1: now also U4.21 (I10); no longer U4.16 (I15)
- net MC11: now also U4.9 (I0); no longer U4.4 (I5)
- net MC12: now also U4.8 (I1); no longer U4.5 (I4)
- net MC13: now also U4.7 (I2); no longer U4.6 (I3)
- net MC14: now also U4.6 (I3); no longer U4.7 (I2)
- net MC15: now also U4.5 (I4); no longer U4.8 (I1)
- net MC16: now also U4.4 (I5); no longer U4.9 (I0)
- net MC2: now also U4.20 (I11); no longer U4.17 (I14)
- net MC3: now also U4.19 (I12); no longer U4.18 (I13)
- net MC4: now also U4.18 (I13); no longer U4.19 (I12)
- net MC5: now also U4.17 (I14); no longer U4.20 (I11)
- net MC6: now also U4.16 (I15); no longer U4.21 (I10)
- net MD1: now also U5.4 (I5); no longer U5.9 (I0)
- net MD11: now also U5.16 (I15); no longer U5.21 (I10)
- net MD12: now also U5.17 (I14); no longer U5.20 (I11)
- net MD13: now also U5.18 (I13); no longer U5.19 (I12)
- net MD14: now also U5.19 (I12); no longer U5.18 (I13)
- net MD15: now also U5.20 (I11); no longer U5.17 (I14)
- net MD16: now also U5.21 (I10); no longer U5.16 (I15)
- net MD2: now also U5.5 (I4); no longer U5.8 (I1)
- net MD3: now also U5.6 (I3); no longer U5.7 (I2)
- net MD4: now also U5.7 (I2); no longer U5.6 (I3)
- net MD5: now also U5.8 (I1); no longer U5.5 (I4)
- net MD6: now also U5.9 (I0); no longer U5.4 (I5)

Commit message: input port
Connections:
- net 3.3V: now also U3.4 (OUT+); no longer U3.3 (OUT-)
- net 5V: now also U3.2 (IN+); no longer U3.1 (IN-)
- net GND: now also U3.1 (IN-), U3.3 (OUT-); no longer U3.2 (IN+), U3.4 (OUT+)
- net S0: now also J2.4 (Pin_4); no longer J2.2 (Pin_2)
- net S1: now also J2.5 (Pin_5); no longer J2.3 (Pin_3)
- net S2: now also J2.6 (Pin_6); no longer J2.4 (Pin_4)
- net S3: now also J2.7 (Pin_7); no longer J2.5 (Pin_5)
- net SCL: now also J2.2 (Pin_2); no longer J2.7 (Pin_7)
- net SDA: now also J2.3 (Pin_3); no longer J2.6 (Pin_6)
Changed lines of the file:
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@@
 	(wire
 		(pts
-			(xy 378.46 242.57) (xy 353.06 242.57)
+			(xy 353.06 242.57) (xy 379.73 242.57)
 		)
 		(stroke
@@
 	(wire
 		(pts
-			(xy 379.73 245.11) (xy 379.73 187.96)
+			(xy 379.73 242.57) (xy 379.73 187.96)
 		)
 		(stroke
@@
 	(wire
 		(pts
-			(xy 378.46 245.11) (xy 378.46 242.57)
-		)
-		(stroke
-			(width 0)
-			(type default)
-		)
-	)
-	(wire
-		(pts
 			(xy 113.03 182.88) (xy 113.03 204.47)
 		)
@@
 		)
 	)
-	(wire
-		(pts
-			(xy 378.46 245.11) (xy 379.73 245.11)
-		)
-		(stroke
-			(width 0)
-			(type default)
-		)
-	)
 	(label "ADDR → GND (for address 0x48)"
 		(at 403.86 194.31 0)
@@
 	(global_label "S2"
 		(shape input)
-		(at 394.97 269.24 90)
+		(at 400.05 269.24 90)
 		(fields_autoplaced yes)
 		(effects
@@
 		)
 		(property "Intersheetrefs" "${INTERSHEET_REFS}"
-			(at 394.97 263.8358 90)
+			(at 400.05 263.8358 90)
 			(effects
 				(font
@@
 	(global_label "S0"
 		(shape input)
-		(at 389.89 269.24 90)
+		(at 394.97 269.24 90)
 		(fields_autoplaced yes)
 		(effects
@@
 		)
 		(property "Intersheetrefs" "${INTERSHEET_REFS}"
-			(at 389.89 263.8358 90)
+			(at 394.97 263.8358 90)
 			(effects
 				(font
@@
 	(global_label "5V"
 		(shape input)
-		(at 398.78 234.95 180)
+		(at 398.78 238.76 180)
 		(fields_autoplaced yes)
 		(effects
@@
 		)
 		(property "Intersheetrefs" "${INTERSHEET_REFS}"
-			(at 393.4967 234.95 0)
+			(at 393.4967 238.76 0)
 			(effects
 				(font
@@
 	(global_label "SCL"
 		(shape input)
-		(at 402.59 269.24 90)
+		(at 389.89 269.24 90)
 		(fields_autoplaced yes)
 		(effects
@@
 		)
 		(property "Intersheetrefs" "${INTERSHEET_REFS}"
-			(at 402.59 262.7472 90)
+			(at 389.89 262.7472 90)
 			(effects
 				(font
@@
 	(global_label "S1"
 		(shape input)
-		(at 392.43 269.24 90)
+		(at 397.51 269.24 90)
 		(fields_autoplaced yes)
 		(effects
@@
 		)
 		(property "Intersheetrefs" "${INTERSHEET_REFS}"
-			(at 392.43 263.8358 90)
+			(at 397.51 263.8358 90)
 			(effects
 				(font
@@
 	(global_label "GND"
 		(shape input)
-		(at 416.56 238.76 0)
+		(at 416.56 234.95 0)
 		(fields_autoplaced yes)
 		(effects
@@
 		)
 		(property "Intersheetrefs" "${INTERSHEET_REFS}"
-			(at 423.4157 238.76 0)
+			(at 423.4157 234.95 0)
 			(effects
 				(font
@@
 	(global_label "S3"
 		(shape input)
-		(at 397.51 269.24 90)
+		(at 402.59 269.24 90)
 		(fields_autoplaced yes)
 		(effects
@@
 		)
 		(property "Intersheetrefs" "${INTERSHEET_REFS}"
-			(at 397.51 263.8358 90)
+			(at 402.59 263.8358 90)
 			(effects
 				(font
@@
 	(global_label "GND"
 		(shape input)
-		(at 398.78 238.76 180)
+		(at 398.78 234.95 180)
 		(fields_autoplaced yes)
 		(effects
@@
 		)
 		(property "Intersheetrefs" "${INTERSHEET_REFS}"
-			(at 391.9243 238.76 0)
+			(at 391.9243 234.95 0)
 			(effects
 				(font
@@
 	(global_label "3.3V"
 		(shape input)
-		(at 416.56 234.95 0)
+		(at 416.56 238.76 0)
 		(fields_autoplaced yes)
 		(effects
@@
 		)
 		(property "Intersheetrefs" "${INTERSHEET_REFS}"
-			(at 423.6576 234.95 0)
+			(at 423.6576 238.76 0)
 			(effects
 				(font
@@
 	(global_label "SDA"
 		(shape input)
-		(at 400.05 269.24 90)
+		(at 392.43 269.24 90)
 		(fields_autoplaced yes)
 		(effects
@@
 		)
 		(property "Intersheetrefs" "${INTERSHEET_REFS}"
-			(at 400.05 262.6867 90)
+			(at 392.43 262.6867 90)
 			(effects
 				(font
