File: kicad/Chess.kicad_pcb (KiCad board)
At the start: 2 copper layers, 238 x 238 mm, 0 parts

Commit message: positions
Parts:
- added J2: Conn_01x08_Pin, Connector_PinHeader_2.54mm:PinHeader_1x08_P2.54mm_Vertical, B.Cu at (146.5, 265.5)
- added U1: CD74HC4067M, MagChess Footprints:CD74HC4067, B.Cu at (69.0, 87.0)
- added U12: A1302xUA, MagChess Footprints:SS49E, F.Cu at (268.0, 135.0)
- added U13: A1302xUA, MagChess Footprints:SS49E, F.Cu at (268.0, 103.0)
- added U14: A1302xUA, MagChess Footprints:SS49E, F.Cu at (268.0, 71.0)
- added U15: A1302xUA, MagChess Footprints:SS49E, F.Cu at (268.0, 39.0)
- added U16: A1302xUA, MagChess Footprints:SS49E, F.Cu at (268.0, 263.0)
- added U17: A1302xUA, MagChess Footprints:SS49E, F.Cu at (268.0, 231.0)
- added U18: A1302xUA, MagChess Footprints:SS49E, F.Cu at (268.0, 199.0)
- added U19: A1302xUA, MagChess Footprints:SS49E, F.Cu at (268.0, 167.0)
- added U2: ADS1015IDGS, MagChess Footprints:ADS1015, B.Cu at (156.0, 119.0)
- added U20: A1302xUA, MagChess Footprints:SS49E, F.Cu at (236.0, 135.0)
- added U21: A1302xUA, MagChess Footprints:SS49E, F.Cu at (236.0, 103.0)
- added U22: A1302xUA, MagChess Footprints:SS49E, F.Cu at (236.0, 71.0)
- added U23: A1302xUA, MagChess Footprints:SS49E, F.Cu at (236.0, 39.0)
- added U24: A1302xUA, MagChess Footprints:SS49E, F.Cu at (236.0, 263.0)
- added U25: A1302xUA, MagChess Footprints:SS49E, F.Cu at (236.0, 231.0)
- added U26: A1302xUA, MagChess Footprints:SS49E, F.Cu at (236.0, 199.0)
- added U27: A1302xUA, MagChess Footprints:SS49E, F.Cu at (236.0, 167.0)
- added U28: A1302xUA, MagChess Footprints:SS49E, F.Cu at (204.0, 135.0)
- added U29: A1302xUA, MagChess Footprints:SS49E, F.Cu at (172.0, 135.0)
- added U3: MP1584EN, MagChess Footprints:MP1584, B.Cu at (155.8, 181.9)
- added U30: A1302xUA, MagChess Footprints:SS49E, F.Cu at (140.0, 135.0)
- added U31: A1302xUA, MagChess Footprints:SS49E, F.Cu at (204.0, 103.0)
- added U32: A1302xUA, MagChess Footprints:SS49E, F.Cu at (172.0, 103.0)
- added U33: A1302xUA, MagChess Footprints:SS49E, F.Cu at (140.0, 103.0)
- added U34: A1302xUA, MagChess Footprints:SS49E, F.Cu at (204.0, 71.0)
- added U35: A1302xUA, MagChess Footprints:SS49E, F.Cu at (172.0, 71.0)
- added U36: A1302xUA, MagChess Footprints:SS49E, F.Cu at (140.0, 71.0)
- added U37: A1302xUA, MagChess Footprints:SS49E, F.Cu at (204.0, 39.0)
- added U38: A1302xUA, MagChess Footprints:SS49E, F.Cu at (172.0, 39.0)
- added U39: A1302xUA, MagChess Footprints:SS49E, F.Cu at (140.0, 39.0)
- added U4: CD74HC4067M, MagChess Footprints:CD74HC4067, B.Cu at (68.6, 215.0)
- added U40: A1302xUA, MagChess Footprints:SS49E, F.Cu at (204.0, 263.0)
- added U41: A1302xUA, MagChess Footprints:SS49E, F.Cu at (172.0, 263.0)
- added U42: A1302xUA, MagChess Footprints:SS49E, F.Cu at (140.0, 263.0)
- added U43: A1302xUA, MagChess Footprints:SS49E, F.Cu at (204.0, 231.0)
- added U44: A1302xUA, MagChess Footprints:SS49E, F.Cu at (172.0, 231.0)
- added U45: A1302xUA, MagChess Footprints:SS49E, F.Cu at (140.0, 231.0)
- added U46: A1302xUA, MagChess Footprints:SS49E, F.Cu at (204.0, 199.0)
- added U47: A1302xUA, MagChess Footprints:SS49E, F.Cu at (172.0, 199.0)
- added U48: A1302xUA, MagChess Footprints:SS49E, F.Cu at (140.0, 199.0)
- added U49: A1302xUA, MagChess Footprints:SS49E, F.Cu at (204.0, 167.0)
- added U5: CD74HC4067M, MagChess Footprints:CD74HC4067, B.Cu at (243.4, 215.0)
- added U50: A1302xUA, MagChess Footprints:SS49E, F.Cu at (172.0, 167.0)
- added U51: A1302xUA, MagChess Footprints:SS49E, F.Cu at (140.0, 167.0)
- added U52: A1302xUA, MagChess Footprints:SS49E, F.Cu at (108.0, 135.0)
- added U53: A1302xUA, MagChess Footprints:SS49E, F.Cu at (76.0, 135.0)
- added U54: A1302xUA, MagChess Footprints:SS49E, F.Cu at (44.0, 135.0)
- added U55: A1302xUA, MagChess Footprints:SS49E, F.Cu at (108.0, 103.0)
- added U56: A1302xUA, MagChess Footprints:SS49E, F.Cu at (76.0, 103.0)
- added U57: A1302xUA, MagChess Footprints:SS49E, F.Cu at (44.0, 103.0)
- added U58: A1302xUA, MagChess Footprints:SS49E, F.Cu at (108.0, 71.0)
- added U59: A1302xUA, MagChess Footprints:SS49E, F.Cu at (76.0, 71.0)
- added U6: CD74HC4067M, MagChess Footprints:CD74HC4067, B.Cu at (244.0, 87.0)
- added U60: A1302xUA, MagChess Footprints:SS49E, F.Cu at (44.0, 71.0)
- added U61: A1302xUA, MagChess Footprints:SS49E, F.Cu at (108.0, 39.0)
- added U62: A1302xUA, MagChess Footprints:SS49E, F.Cu at (76.0, 39.0)
- added U63: A1302xUA, MagChess Footprints:SS49E, F.Cu at (44.0, 39.0)
- added U64: A1302xUA, MagChess Footprints:SS49E, F.Cu at (108.0, 263.0)
- added U65: A1302xUA, MagChess Footprints:SS49E, F.Cu at (76.0, 263.0)
- added U66: A1302xUA, MagChess Footprints:SS49E, F.Cu at (44.0, 263.0)
- added U67: A1302xUA, MagChess Footprints:SS49E, F.Cu at (108.0, 231.0)
- added U68: A1302xUA, MagChess Footprints:SS49E, F.Cu at (76.0, 231.0)
- added U69: A1302xUA, MagChess Footprints:SS49E, F.Cu at (44.0, 231.0)
- added U70: A1302xUA, MagChess Footprints:SS49E, F.Cu at (108.0, 199.0)
- added U71: A1302xUA, MagChess Footprints:SS49E, F.Cu at (76.0, 199.0)
- added U72: A1302xUA, MagChess Footprints:SS49E, F.Cu at (44.0, 199.0)
- added U73: A1302xUA, MagChess Footprints:SS49E, F.Cu at (108.0, 167.0)
- added U74: A1302xUA, MagChess Footprints:SS49E, F.Cu at (76.0, 167.0)
- added U75: A1302xUA, MagChess Footprints:SS49E, F.Cu at (44.0, 167.0)
