File: kicad/Chess.kicad_pcb (KiCad board)
At the start: 2 copper layers, 238 x 238 mm, 71 parts, among them J2 Conn_01x08_Pin, U1 CD74HC4067M, U12 A1302xUA, U13 A1302xUA, U14 A1302xUA, U15 A1302xUA, U16 A1302xUA, U17 A1302xUA, U18 A1302xUA, U19 A1302xUA, U2 ADS1015IDGS, U20 A1302xUA, U21 A1302xUA, U22 A1302xUA, U23 A1302xUA, U24 A1302xUA, U25 A1302xUA, U26 A1302xUA, U27 A1302xUA, U28 A1302xUA, U29 A1302xUA, U3 MP1584EN, U30 A1302xUA, U31 A1302xUA, U32 A1302xUA, U33 A1302xUA, U34 A1302xUA, U35 A1302xUA, U36 A1302xUA, U37 A1302xUA, U38 A1302xUA, U39 A1302xUA, U4 CD74HC4067M, U40 A1302xUA, U41 A1302xUA, U42 A1302xUA, U43 A1302xUA, U44 A1302xUA, U45 A1302xUA, U46 A1302xUA, U47 A1302xUA, U48 A1302xUA, U49 A1302xUA, U5 CD74HC4067M, U50 A1302xUA, U51 A1302xUA, U52 A1302xUA, U53 A1302xUA, U54 A1302xUA, U55 A1302xUA, U56 A1302xUA, U57 A1302xUA, U58 A1302xUA, U59 A1302xUA, U6 CD74HC4067M, U60 A1302xUA, U61 A1302xUA, U62 A1302xUA, U63 A1302xUA, U64 A1302xUA, U65 A1302xUA, U66 A1302xUA, U67 A1302xUA, U68 A1302xUA, U69 A1302xUA, U70 A1302xUA, U71 A1302xUA, U72 A1302xUA, U73 A1302xUA, U74 A1302xUA, U75 A1302xUA

Commit message: routes 1
Parts:
- moved J2 2.50 mm to (146.5, 263.0)
- moved U1 2.00 mm to (67.0, 87.0)
- moved U4 1.60 mm to (67.0, 215.0)
- moved U5 1.60 mm to (245.0, 215.0)
- moved U6 1.00 mm to (245.0, 87.0)
Routing:
- net GND: track 0.00 -> 2247.5 mm
- net 3.3V: track 0.00 -> 2222.2 mm
- net Net-(U2-AIN2): track 0.00 -> 166.0 mm, vias 0 -> 4
- net SDA: track 0.00 -> 164.4 mm
- net SCL: track 0.00 -> 164.0 mm
- net Net-(U2-AIN3): track 0.00 -> 129.5 mm, vias 0 -> 2
- net MA4: track 0.00 -> 110.5 mm
- net MD4: track 0.00 -> 110.5 mm
- net MA13: track 0.00 -> 108.0 mm
- net MD13: track 0.00 -> 108.0 mm
- net MB4: track 0.00 -> 105.9 mm
- net MC4: track 0.00 -> 105.9 mm
- net MB13: track 0.00 -> 104.5 mm
- net MC13: track 0.00 -> 104.5 mm
- net Net-(U1-COM): track 0.00 -> 103.9 mm, vias 0 -> 2
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
Commit message: routes 2
Parts:
- moved U3 2.04 mm to (155.8, 183.9)
- moved U2 0.81 mm to (156.0, 118.2), turned to 180 degrees
Connections:
- J2 pad 6: SCL -> SDA
- J2 pad 7: SDA -> SCL
- U4 pad 1: Net-(U2-AIN2) -> Net-(U2-AIN3)
- U5 pad 1: Net-(U2-AIN3) -> Net-(U2-AIN2)
Routing:
- net S3: track 0.00 -> 563.1 mm, vias 0 -> 8
- net S2: track 0.00 -> 554.6 mm, vias 0 -> 8
- net S1: track 0.00 -> 540.1 mm, vias 0 -> 8
- net S0: track 0.00 -> 525.9 mm, vias 0 -> 7
- net 3.3V: track 2222.2 -> 2110.3 mm
- net Net-(U2-AIN3): track 129.5 -> 175.6 mm, vias 2 -> 0
- net GND: track 2247.5 -> 2211.1 mm
- net Net-(U2-AIN2): track 166.0 -> 180.8 mm, vias 4 -> 2
- net SCL: track 164.0 -> 152.6 mm
- net 5V: track 83.7 -> 94.8 mm
- net SDA: track 164.4 -> 153.9 mm
- net Net-(U2-AIN0): track 103.4 -> 113.3 mm
- net MD11: track 52.8 -> 61.6 mm
- net MC11: track 51.3 -> 59.5 mm
- net MB6: track 54.9 -> 63.1 mm
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
Commit message: fill zone
Routing:
- added copper zone on B.Cu, net (none)
- added copper zone on F.Cu, net (none)
Changed lines of the file:
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@@
 		(layer "User.2")
 	)
+	(gr_circle
+		(center 155 214)
+		(end 171 214)
+		(stroke
+			(width 0.1)
+			(type default)
+		)
+		(fill no)
+		(layer "User.3")
+	)
+	(gr_circle
+		(center 219 150)
+		(end 235 149)
+		(stroke
+			(width 0.1)
+			(type default)
+		)
+		(fill no)
+		(layer "User.3")
+	)
+	(gr_circle
+		(center 155 150)
+		(end 171 150)
+		(stroke
+			(width 0.1)
+			(type default)
+		)
+		(fill no)
+		(layer "User.3")
+	)
+	(gr_circle
+		(center 91 150)
+		(end 107 150)
+		(stroke
+			(width 0.1)
+			(type default)
+		)
+		(fill no)
+		(layer "User.3")
+	)
+	(gr_circle
+		(center 155 86)
+		(end 171 86)
+		(stroke
+			(width 0.1)
+			(type default)
+		)
+		(fill no)
+		(layer "User.3")
+	)
 	(gr_line
 		(start 83 78)
@@
 	)
 	(segment
-		(start 66 91.5)
-		(end 66.69 90.81)
-		(width 0.2)
-		(layer "F.Cu")
-		(net 1)
-	)
-	(segment
-		(start 66.69 90.81)
-		(end 74.6 90.81)
+		(start 66 172)
+		(end 66 130)
 		(width 0.2)
 		(layer "F.Cu")
@@
 	)
 	(segment
-		(start 66 172)
-		(end 66 130)
+		(start 66 170)
+		(end 66 172)
 		(width 0.2)
 		(layer "F.Cu")
@@
 	)
 	(segment
-		(start 66 170)
-		(end 66 172)
+		(start 66 90.81)
+		(end 74.6 90.81)
 		(width 0.2)
 		(layer "F.Cu")
@@
 	)
 	(via
-		(at 66 91.5)
+		(at 66 90.81)
 		(size 0.6)
 		(drill 0.3)
@@
 	)
 	(segment
-		(start 246 211.19)
-		(end 246 249)
+		(start 66 130)
+		(end 66 90.81)
 		(width 0.2)
 		(layer "B.Cu")
@@
 	)
 	(segment
-		(start 66 130)
-		(end 66 91.5)
+		(start 246 211.19)
+		(end 246 249)
 		(width 0.2)
 		(layer "B.Cu")
@@
 	)
 	(segment
-		(start 70.77 85.73)
-		(end 74.6 85.73)
-		(width 0.2)
-		(layer "B.Cu")
-		(net 5)
-	)
-	(segment
 		(start 242 247)
 		(end 149 247)
@@
 	)
 	(segment
-		(start 70 86.5)
-		(end 70.77 85.73)
-		(width 0.2)
-		(layer "B.Cu")
-		(net 5)
-	)
-	(segment
 		(start 70 130)
-		(end 70 86.5)
+		(end 70 85.73)
 		(width 0.2)
 		(layer "B.Cu")
@@
 	)
 	(segment
-		(start 68.73 88.27)
-		(end 74.6 88.27)
+		(start 70 85.73)
+		(end 74.6 85.73)
 		(width 0.2)
-		(layer "F.Cu")
-		(net 6)
+		(layer "B.Cu")
+		(net 5)
 	)
 	(segment
@@
 	)
 	(segment
-		(start 68 170)
-		(end 68 171)
+		(start 68 88.27)
+		(end 74.6 88.27)
 		(width 0.2)
 		(layer "F.Cu")
@@
 	)
 	(segment
-		(start 68 89)
-		(end 68.73 88.27)
+		(start 68 170)
+		(end 68 171)
 		(width 0.2)
 		(layer "F.Cu")
@@
 	)
 	(via
-		(at 68 89)
+		(at 68 88.27)
 		(size 0.6)
 		(drill 0.3)
@@
 	)
 	(segment
+		(start 68 130)
+		(end 68 88.27)
+		(width 0.2)
+		(layer "B.Cu")
+		(net 6)
+	)
+	(segment
 		(start 244 213.73)
 		(end 244 248)
@@
 	)
 	(segment
-		(start 68 130)
-		(end 68 89)
-		(width 0.2)
-		(layer "B.Cu")
-		(net 6)
-	)
-	(segment
 		(start 244 248)
 		(end 243 249)
@@
 	)
 	(segment
-		(start 64 170)
-		(end 64 130)
+		(start 64 93.35)
+		(end 74.6 93.35)
 		(width 0.2)
 		(layer "F.Cu")
@@
 	)
 	(segment
-		(start 64 94)
-		(end 64.65 93.35)
+		(start 64 170)
+		(end 64 130)
 		(width 0.2)
 		(layer "F.Cu")
@@
 	)
 	(segment
-		(start 64.65 93.35)
-		(end 74.6 93.35)
-		(width 0.2)
-		(layer "F.Cu")
-		(net 7)
-	)
-	(segment
 		(start 64 221.35)
 		(end 74.6 221.35)
@@
 	)
 	(via
-		(at 64 94)
+		(at 64 93.35)
 		(size 0.6)
 		(drill 0.3)
@@
 	(segment
 		(start 64 130)
-		(end 64 94)
+		(end 64 93.35)
 		(width 0.2)
 		(layer "B.Cu")
@@
 		(net 78)
 	)
+	(zone
+		(net 0)
+		(net_name "")
+		(layers "F.Cu" "B.Cu")
+		(hatch edge 0.5)
+		(connect_pads
+			(clearance 0.5)
+		)
+		(min_thickness 0.25)
+		(filled_areas_thickness no)
+		(fill
+			(thermal_gap 0.5)
+			(thermal_bridge_width 0.5)
+			(island_removal_mode 1)
+			(island_area_min 10)
+		)
+		(polygon
+			(pts
+				(xy 30 25) (xy 280 25) (xy 280 275) (xy 30 275)
+			)
+		)
+	)
 	(embedded_fonts no)

Commit message: routing v2
Parts:
- moved U1 7.00 mm to (60.0, 87.0)
- moved U4 7.00 mm to (60.0, 215.0)
- moved U5 5.00 mm to (250.0, 215.0)
- moved U6 5.00 mm to (250.0, 87.0)
- moved J2 2.00 mm to (146.5, 265.0)
Connections:
- U1 pad 16: MB1 -> MB6
- U1 pad 17: MB2 -> MB5
- U1 pad 18: MB3 -> MB4
- U1 pad 19: MB4 -> MB3
- U1 pad 20: MB5 -> MB2
- U1 pad 21: MB6 -> MB1
- U1 pad 4: MB11 -> MB16
- U1 pad 5: MB12 -> MB15
- U1 pad 6: MB13 -> MB14
- U1 pad 7: MB14 -> MB13
- U1 pad 8: MB15 -> MB12
- U1 pad 9: MB16 -> MB11
- U4 pad 16: MC1 -> MC6
- U4 pad 17: MC2 -> MC5
- U4 pad 18: MC3 -> MC4
- U4 pad 19: MC4 -> MC3
- U4 pad 20: MC5 -> MC2
- U4 pad 21: MC6 -> MC1
- U4 pad 4: MC11 -> MC16
- U4 pad 5: MC12 -> MC15
- U4 pad 6: MC13 -> MC14
- U4 pad 7: MC14 -> MC13
- U4 pad 8: MC15 -> MC12
- U4 pad 9: MC16 -> MC11
- U5 pad 16: MD16 -> MD11
- U5 pad 17: MD15 -> MD12
- U5 pad 18: MD14 -> MD13
- U5 pad 19: MD13 -> MD14
- U5 pad 20: MD12 -> MD15
- U5 pad 21: MD11 -> MD16
- U5 pad 4: MD6 -> MD1
- U5 pad 5: MD5 -> MD2
- U5 pad 6: MD4 -> MD3
- U5 pad 7: MD3 -> MD4
- U5 pad 8: MD2 -> MD5
- U5 pad 9: MD1 -> MD6
- U6 pad 16: MA16 -> MA11
- U6 pad 17: MA15 -> MA12
- U6 pad 18: MA14 -> MA13
- U6 pad 19: MA13 -> MA14
- U6 pad 20: MA12 -> MA15
- U6 pad 21: MA11 -> MA16
- U6 pad 4: MA6 -> MA1
- U6 pad 5: MA5 -> MA2
- U6 pad 6: MA4 -> MA3
- U6 pad 7: MA3 -> MA4
- U6 pad 8: MA2 -> MA5
- U6 pad 9: MA1 -> MA6
Routing:
- net 3.3V: track 2110.3 -> 2215.6 mm, vias 0 -> 2
- net GND: track 2211.1 -> 2312.8 mm
- net MD11: track 61.6 -> 44.3 mm
- net MA11: track 52.8 -> 36.8 mm
- net MC11: track 59.5 -> 44.2 mm
- net S3: track 563.5 -> 548.2 mm, vias 8 -> 9
- net MA6: track 66.7 -> 51.6 mm
- net MB11: track 51.3 -> 36.2 mm
- net S2: track 555.0 -> 541.2 mm, vias 8 -> 9
- net MB6: track 63.1 -> 50.3 mm
- net MD12: track 80.0 -> 67.7 mm
- net MA12: track 80.0 -> 67.7 mm
- net MD5: track 82.5 -> 70.9 mm
- net MA5: track 82.5 -> 70.9 mm
- net MB1: track 15.3 -> 26.5 mm
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
Commit message: input port
Parts:
- moved J2 17.8 mm to (164.2, 265.0), turned to 90 degrees
- turned U3 to 180 degrees
Connections:
- J2 pad 2: S0 -> SCL
- J2 pad 3: S1 -> SDA
- J2 pad 4: S2 -> S0
- J2 pad 5: S3 -> S1
- J2 pad 6: SDA -> S2
- J2 pad 7: SCL -> S3
- U3 pad 1: 5V -> GND
- U3 pad 2: GND -> 5V
- U3 pad 3: 3.3V -> GND
- U3 pad 4: GND -> 3.3V
Routing:
- net 5V: track 96.8 -> 83.4 mm

Commit message: PSU remake
Parts:
- moved U3 2.04 mm to (155.0, 182.0)
Routing:
- net Net-(U2-AIN2): track 188.7 -> 181.3 mm
- net GND: track 2312.8 -> 2306.0 mm
- net Net-(U2-AIN3): track 182.6 -> 176.1 mm
- net MD11: track 44.3 -> 46.8 mm
- net MC11: track 44.2 -> 46.7 mm
- net 3.3V: track 2215.9 -> 2215.0 mm
- net SCL: track 154.6 -> 155.4 mm
- net SDA: track 155.9 -> 156.7 mm
- net 5V: track 83.4 -> 83.9 mm

Commit message: cleanup
Routing:
- net SDA: track 156.7 -> 155.7 mm
Changed lines of the file:
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@@
+	)
+	(segment
+		(start 161.7 232.9)
+		(end 168.4 226.2)
+		(width 0.2)
+		(layer "F.Cu")
+		(net 2)
+	)
+	(segment
+		(start 168.4 226.2)
+		(end 168.4 206.4)
+		(width 0.2)
+		(layer "F.Cu")
+		(net 2)
 	)
 	(segment
@@
 	)
 	(segment
+		(start 168.4 206.4)
+		(end 161 199)
+		(width 0.2)
+		(layer "F.Cu")
+		(net 2)
+	)
+	(segment
+		(start 169 159)
+		(end 169 141)
+		(width 0.2)
+		(layer "F.Cu")
+		(net 2)
+	)
+	(segment
+		(start 161.7 265)
+		(end 161.7 232.9)
+		(width 0.2)
+		(layer "F.Cu")
+		(net 2)
+	)
+	(segment
 		(start 161 199)
 		(end 161 167)
@@
 	)
 	(segment
-		(start 169 207)
-		(end 161 199)
-		(width 0.2)
-		(layer "F.Cu")
-		(net 2)
-	)
-	(segment
-		(start 169 226.125)
-		(end 169 207)
-		(width 0.2)
-		(layer "F.Cu")
-		(net 2)
-	)
-	(segment
-		(start 161.7 233.425)
-		(end 169 226.125)
-		(width 0.2)
-		(layer "F.Cu")
-		(net 2)
-	)
-	(segment
-		(start 161.7 265)
-		(end 161.7 233.425)
-		(width 0.2)
-		(layer "F.Cu")
-		(net 2)
-	)
-	(segment
-		(start 169 159)
-		(end 169 141)
-		(width 0.2)
-		(layer "F.Cu")
-		(net 2)
-	)
-	(segment
 		(start 73.89 206.11)
 		(end 76 204)
@@
 	)
 	(segment
+		(start 159.16 233.055365)
+		(end 159.16 265)
+		(width 0.2)
+		(layer "F.Cu")
+		(net 4)
+	)
+	(segment
+		(start 159.81 122)
+		(end 159.81 134.81)
+		(width 0.2)
+		(layer "F.Cu")
+		(net 4)
+	)
+	(segment
+		(start 159 166)
+		(end 159 199)
+		(width 0.2)
+		(layer "F.Cu")
+		(net 4)
+	)
+	(segment
+		(start 167 142)
+		(end 167 158)
+		(width 0.2)
+		(layer "F.Cu")
+		(net 4)
+	)
+	(segment
 		(start 159.81 134.81)
 		(end 167 142)
@@
 	)
 	(segment
-		(start 159.81 122)
-		(end 159.81 134.81)
-		(width 0.2)
-		(layer "F.Cu")
-		(net 4)
-	)
-	(segment
-		(start 159 166)
-		(end 159 199)
-		(width 0.2)
-		(layer "F.Cu")
-		(net 4)
-	)
-	(segment
-		(start 168 225.320001)
-		(end 159.16 234.160001)
-		(width 0.2)
-		(layer "F.Cu")
-		(net 4)
-	)
-	(segment
-		(start 168 208)
-		(end 168 225.320001)
-		(width 0.2)
-		(layer "F.Cu")
-		(net 4)
-	)
-	(segment
-		(start 159 199)
-		(end 168 208)
-		(width 0.2)
-		(layer "F.Cu")
-		(net 4)
-	)
-	(segment
-		(start 167 142)
-		(end 167 158)
+		(start 166.8 206.8)
+		(end 166.8 225.415365)
 		(width 0.2)
 		(layer "F.Cu")
@@
 	)
 	(segment
-		(start 159.16 234.160001)
-		(end 159.16 265)
+		(start 159 199)
+		(end 166.8 206.8)
+		(width 0.2)
+		(layer "F.Cu")
+		(net 4)
+	)
+	(segment
+		(start 166.8 225.415365)
+		(end 159.16 233.055365)
 		(width 0.2)
 		(layer "F.Cu")
@@
 	)
 	(segment
+		(start 164.24 232.76)
+		(end 164.24 265)
+		(width 0.2)
+		(layer "F.Cu")
+		(net 8)
+	)
+	(segment
+		(start 164.25 200.25)
+		(end 170 206)
+		(width 0.2)
+		(layer "F.Cu")
+		(net 8)
+	)
+	(segment
 		(start 164.25 188.4)
 		(end 164.25 200.25)
@@
 		(width 0.2)
 		(layer "F.Cu")
-		(net 8)
-	)
-	(segment
-		(start 164.25 200.25)
-		(end 170 206)
-		(width 0.2)
-		(layer "F.Cu")
-		(net 8)
-	)
-	(segment
-		(start 164.24 232.76)
-		(end 164.24 265)
-		(width 0.2)
-		(layer "F.Cu")
