File: kicad/Chess.kicad_pcb (KiCad board)
At the start: 2 copper layers, 238 x 238 mm, 71 parts, among them J2 Conn_01x08_Pin, U1 CD74HC4067M, U12 A1302xUA, U13 A1302xUA, U14 A1302xUA, U15 A1302xUA, U16 A1302xUA, U17 A1302xUA, U18 A1302xUA, U19 A1302xUA, U2 ADS1015IDGS, U20 A1302xUA, U21 A1302xUA, U22 A1302xUA, U23 A1302xUA, U24 A1302xUA, U25 A1302xUA, U26 A1302xUA, U27 A1302xUA, U28 A1302xUA, U29 A1302xUA, U3 MP1584EN, U30 A1302xUA, U31 A1302xUA, U32 A1302xUA, U33 A1302xUA, U34 A1302xUA, U35 A1302xUA, U36 A1302xUA, U37 A1302xUA, U38 A1302xUA, U39 A1302xUA, U4 CD74HC4067M, U40 A1302xUA, U41 A1302xUA, U42 A1302xUA, U43 A1302xUA, U44 A1302xUA, U45 A1302xUA, U46 A1302xUA, U47 A1302xUA, U48 A1302xUA, U49 A1302xUA, U5 CD74HC4067M, U50 A1302xUA, U51 A1302xUA, U52 A1302xUA, U53 A1302xUA, U54 A1302xUA, U55 A1302xUA, U56 A1302xUA, U57 A1302xUA, U58 A1302xUA, U59 A1302xUA, U6 CD74HC4067M, U60 A1302xUA, U61 A1302xUA, U62 A1302xUA, U63 A1302xUA, U64 A1302xUA, U65 A1302xUA, U66 A1302xUA, U67 A1302xUA, U68 A1302xUA, U69 A1302xUA, U70 A1302xUA, U71 A1302xUA, U72 A1302xUA, U73 A1302xUA, U74 A1302xUA, U75 A1302xUA

Commit message: cleanup
Routing:
- net MD6: track 52.7 -> 40.4 mm
- net MC6: track 51.1 -> 39.8 mm
- net MD11: track 46.8 -> 48.6 mm
Changed lines of the file:
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@@
+	)
+	(segment
+		(start 45.796051 170)
+		(end 45.796051 165.203949)
+		(width 0.2)
+		(layer "F.Cu")
+		(net 14)
 	)
 	(segment
@@
 		(start 239.65 93.35)
 		(end 237.796051 95.203949)
-		(width 0.2)
-		(layer "F.Cu")
-		(net 14)
-	)
-	(segment
-		(start 45.796051 180)
-		(end 45.796051 165.203949)
 		(width 0.2)
 		(layer "F.Cu")
@@
 	)
 	(via
-		(at 45.796051 180)
+		(at 45.796051 170)
 		(size 0.6)
 		(drill 0.3)
@@
 	)
 	(segment
-		(start 45.796051 180)
-		(end 45.796051 197.203949)
-		(width 0.2)
-		(layer "B.Cu")
-		(net 14)
-	)
-	(segment
 		(start 45.796051 261.203949)
 		(end 141.796051 261.203949)
@@
 		(start 45.796051 37.203949)
 		(end 269.796051 37.203949)
+		(width 0.2)
+		(layer "B.Cu")
+		(net 14)
+	)
+	(segment
+		(start 45.796051 170)
+		(end 45.796051 197.203949)
 		(width 0.2)
 		(layer "B.Cu")
@@
 	)
 	(segment
-		(start 52.4 262.4)
+		(start 74.203949 264.796051)
+		(end 52.4 242.992102)
+		(width 0.2)
+		(layer "F.Cu")
+		(net 40)
+	)
+	(segment
+		(start 52.4 242.992102)
 		(end 52.4 234.05)
-		(width 0.2)
-		(layer "F.Cu")
-		(net 40)
-	)
-	(segment
-		(start 54.796051 264.796051)
-		(end 52.4 262.4)
-		(width 0.2)
-		(layer "F.Cu")
-		(net 40)
-	)
-	(segment
-		(start 74.203949 264.796051)
-		(end 54.796051 264.796051)
 		(width 0.2)
 		(layer "F.Cu")
@@
 	)
 	(segment
-		(start 255.203949 264.796051)
-		(end 257.6 262.4)
+		(start 234.203949 264.796051)
+		(end 234.203949 261.796051)
 		(width 0.2)
 		(layer "F.Cu")
@@
 	)
 	(segment
-		(start 257.6 262.4)
+		(start 234.203949 261.796051)
+		(end 257.6 238.4)
+		(width 0.2)
+		(layer "F.Cu")
+		(net 47)
+	)
+	(segment
+		(start 257.6 238.4)
 		(end 257.6 234.05)
-		(width 0.2)
-		(layer "F.Cu")
-		(net 47)
-	)
-	(segment
-		(start 234.203949 264.796051)
-		(end 255.203949 264.796051)
 		(width 0.2)
 		(layer "F.Cu")
@@
 	)
 	(segment
+		(start 234.203949 168.796051)
+		(end 234.203949 188.203949)
+		(width 0.2)
+		(layer "F.Cu")
+		(net 61)
+	)
+	(segment
 		(start 257.6 191.6)
 		(end 257.6 195.95)
@@
 	)
 	(segment
-		(start 234.203949 168.796051)
-		(end 234.203949 185.203949)
-		(width 0.2)
-		(layer "F.Cu")
-		(net 61)
-	)
-	(segment
 		(start 256 190)
 		(end 257.6 191.6)
@@
 	)
 	(segment
-		(start 234.203949 185.203949)
-		(end 239 190)
+		(start 234.203949 188.203949)
+		(end 236 190)
 		(width 0.2)
 		(layer "F.Cu")
@@
 	)
 	(segment
-		(start 239 190)
+		(start 236 190)
 		(end 256 190)
 		(width 0.2)
@@
 	)
 	(segment
-		(start 237 112)
+		(start 256 112)
+		(end 257.6 110.4)
+		(width 0.2)
+		(layer "F.Cu")
+		(net 63)
+	)
+	(segment
+		(start 236.203949 112)
 		(end 256 112)
 		(width 0.2)
@@
 	)
 	(segment
-		(start 234.203949 114.796051)
-		(end 237 112)
+		(start 234.203949 136.796051)
+		(end 234.203949 114)
 		(width 0.2)
 		(layer "F.Cu")
@@
 	)
 	(segment
-		(start 234.203949 136.796051)
-		(end 234.203949 114.796051)
+		(start 234.203949 114)
+		(end 236.203949 112)
 		(width 0.2)
 		(layer "F.Cu")
@@
 		(width 0.2)
 		(layer "F.Cu")
-		(net 63)
-	)
-	(segment
-		(start 256 112)
-		(end 257.6 110.4)
-		(width 0.2)
-		(layer "F.Cu")

Commit message: ADC footprint
Routing:
- net GND: track 2306.0 -> 2307.4 mm
Changed lines of the file:
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@@
 		)
 		(pad "1" thru_hole roundrect
-			(at -9.25 4.1 180)
+			(at -9.3 4.1 180)
 			(size 1.8 1.8)
 			(drill 1.2)
@@
 		)
 		(pad "1" thru_hole roundrect
-			(at -9.25 6.64 180)
+			(at -9.3 6.7 180)
 			(size 1.8 1.8)
 			(drill 1.2)
@@
 		)
 		(pad "2" thru_hole roundrect
-			(at -9.25 -6.4 180)
+			(at -9.3 -6.7 180)
 			(size 1.8 1.8)
 			(drill 1.2)
@@
 		)
 		(pad "2" thru_hole roundrect
-			(at -9.25 -3.86 180)
+			(at -9.3 -4.1 180)
 			(size 1.8 1.8)
 			(drill 1.2)
@@
 		)
 		(pad "3" thru_hole roundrect
-			(at 9.25 4.1 180)
+			(at 9.4 4.1 180)
 			(size 1.8 1.8)
 			(drill 1.2)
@@
 		)
 		(pad "3" thru_hole roundrect
-			(at 9.25 6.64 180)
+			(at 9.4 6.7 180)
 			(size 1.8 1.8)
 			(drill 1.2)
@@
 		)
 		(pad "4" thru_hole roundrect
-			(at 9.25 -6.4 180)
+			(at 9.4 -6.7 180)
 			(size 1.8 1.8)
 			(drill 1.2)
@@
 		)
 		(pad "4" thru_hole roundrect
-			(at 9.25 -3.86 180)
+			(at 9.4 -4.1 180)
 			(size 1.8 1.8)
 			(drill 1.2)
@@
 	)
 	(segment
+		(start 164.3 175.3)
+		(end 164.3 168.7)
+		(width 0.2)
+		(layer "B.Cu")
+		(net 3)
+	)
+	(segment
 		(start 268 231)
 		(end 268 167)
@@
 	)
 	(segment
-		(start 44 167)
+		(start 144 167)
+		(end 166 167)
+		(width 0.2)
+		(layer "B.Cu")
+		(net 3)
+	)
+	(segment
+		(start 166 167)
 		(end 268 167)
 		(width 0.2)
@@
 	)
 	(segment
+		(start 44 167)
+		(end 144 167)
+		(width 0.2)
+		(layer "B.Cu")
+		(net 3)
+	)
+	(segment
 		(start 237.4 90.81)
 		(end 236 89.41)
@@
 	)
 	(segment
-		(start 145.75 177.9)
-		(end 145.75 175.36)
-		(width 0.2)
-		(layer "B.Cu")
-		(net 3)
-	)
-	(segment
 		(start 242.4 218.81)
 		(end 237.81 218.81)
@@
 	)
 	(segment
-		(start 164.25 175.36)
-		(end 164.25 167)
-		(width 0.2)
-		(layer "B.Cu")
-		(net 3)
-	)
-	(segment
 		(start 268 103)
 		(end 268 39)
@@
 	)
 	(segment
-		(start 164.25 177.9)
-		(end 164.25 175.36)
+		(start 164.3 177.9)
+		(end 164.3 175.3)
 		(width 0.2)
 		(layer "B.Cu")
@@
 	)
 	(segment
+		(start 164.3 168.7)
+		(end 166 167)
+		(width 0.2)
+		(layer "B.Cu")
+		(net 3)
+	)
+	(segment
 		(start 44 135)
 		(end 268 135)
@@
 	)
 	(segment
+		(start 145.6 168.6)
+		(end 144 167)
+		(width 0.2)
+		(layer "B.Cu")
+		(net 3)
+	)
+	(segment
 		(start 204 199)
 		(end 236 199)
@@
 	)
 	(segment
-		(start 145.75 175.36)
-		(end 145.75 167)
+		(start 165.08 122)
+		(end 165.08 103)
 		(width 0.2)
 		(layer "B.Cu")
@@
 	)
 	(segment
-		(start 165.08 122)
-		(end 165.08 103)
+		(start 145.6 177.9)
+		(end 145.6 175.3)
 		(width 0.2)
 		(layer "B.Cu")
@@
 	)
 	(segment
+		(start 145.6 175.3)
+		(end 145.6 168.6)
+		(width 0.2)
+		(layer "B.Cu")
+		(net 3)
+	)
+	(segment
 		(start 237.4 90.81)
 		(end 242.4 90.81)
@@
 	)
 	(segment
-		(start 164.24 232.76)
-		(end 164.24 265)
+		(start 170 206)
+		(end 170 227)
 		(width 0.2)
 		(layer "F.Cu")
@@
 	)
 	(segment
-		(start 164.25 200.25)
-		(end 170 206)
+		(start 170 227)
+		(end 164.24 232.76)
 		(width 0.2)
 		(layer "F.Cu")
@@
 	)
 	(segment
-		(start 164.25 188.4)
+		(start 164.24 232.76)
+		(end 164.24 265)
+		(width 0.2)
+		(layer "F.Cu")
+		(net 8)
+	)
+	(segment
+		(start 164.25 188.75)
 		(end 164.25 200.25)
 		(width 0.2)
@@
 	)
 	(segment
-		(start 170 206)
-		(end 170 227)
+		(start 164.3 188.7)
+		(end 164.3 186.1)
 		(width 0.2)
 		(layer "F.Cu")
@@
 	)
 	(segment
-		(start 170 227)
-		(end 164.24 232.76)
+		(start 164.3 188.7)
+		(end 164.25 188.75)
 		(width 0.2)
 		(layer "F.Cu")
@@
 	)
 	(segment
-		(start 164.25 188.4)
-		(end 164.25 185.86)
+		(start 164.25 200.25)
+		(end 170 206)
 		(width 0.2)
 		(layer "F.Cu")
@@
 	)
 	(segment
+		(start 145.6 188.7)
+		(end 145.6 195.603949)
+		(width 0.2)
+		(layer "B.Cu")
+		(net 14)
+	)
+	(segment
 		(start 74.6 80.65)
 		(end 77.796051 83.846051)
@@
 	)
 	(segment
-		(start 145.75 188.4)
-		(end 145.75 185.86)
-		(width 0.2)
-		(layer "B.Cu")
-		(net 14)
-	)
-	(segment
 		(start 167.43 133.203949)
 		(end 167.43 122)
@@
 	)
 	(segment
-		(start 145.75 188.4)
-		(end 145.75 197.203949)
-		(width 0.2)
-		(layer "B.Cu")
-		(net 14)
-	)
-	(segment
 		(start 109.796051 69.203949)
 		(end 205.796051 69.203949)
@@
 	)
 	(segment
+		(start 144 197.203949)
+		(end 205.796051 197.203949)
+		(width 0.2)
+		(layer "B.Cu")
+		(net 14)
+	)
+	(segment
+		(start 145.6 186.1)
+		(end 145.6 188.7)
+		(width 0.2)
+		(layer "B.Cu")
+		(net 14)
+	)
+	(segment
 		(start 269.796051 261.203949)
 		(end 173.796051 261.203949)
@@
 	(segment
 		(start 109.796051 197.203949)
-		(end 205.796051 197.203949)
+		(end 144 197.203949)
+		(width 0.2)
+		(layer "B.Cu")
+		(net 14)
+	)
+	(segment
+		(start 145.6 195.603949)
+		(end 144 197.203949)
 		(width 0.2)
 		(layer "B.Cu")
