File: kicad/pcb/MagChess.kicad_pcb (KiCad board)
At the start: 2 copper layers, 238 x 238 mm, 71 parts, among them J2 Conn_01x08_Pin, U1 CD74HC4067M, U12 A1302xUA, U13 A1302xUA, U14 A1302xUA, U15 A1302xUA, U16 A1302xUA, U17 A1302xUA, U18 A1302xUA, U19 A1302xUA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

Commit message: parts update
Parts:
- U12, U13, U14, U15, U16, U17, U18, U19, U20, U21, U22, U23, U24, U25, U26, U27, U28, U29, U30, U31, U32, U33, U34, U35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: value A1302xUA -> SS49E
